File: schematics/base/base.kicad_pcb (KiCad board)
At the start: 2 copper layers, 68.6 x 53.3 mm, 20 parts, among them J1 BARREL_JACK, J2 CONN_01X04_FEMALE, J3 CONN_02X04, P1 Power, P2 Analog, P3 Digital, P4 Digital, P5 CONN_01X01, P6 CONN_01X01, P7 CONN_01X01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

Commit message: added schematic for base
Connections:
- Q1 pad 1: Net-(D1-Pad2) -> Net-(Q1-Pad1)
- Q2 pad 1: Net-(D2-Pad2) -> Net-(Q2-Pad1)
- Q3 pad 1: Net-(D3-Pad2) -> Net-(Q3-Pad1)
- R1 pad 1: Net-(D1-Pad2) -> Net-(Q1-Pad1)
- R2 pad 1: Net-(D2-Pad2) -> Net-(Q2-Pad1)
- R3 pad 1: Net-(D3-Pad2) -> Net-(Q3-Pad1)
Routing:
- net Net-(Q3-Pad1): track 0.00 -> 8.13 mm
- net Net-(Q2-Pad1): track 0.00 -> 8.13 mm
- net Net-(Q1-Pad1): track 0.00 -> 8.13 mm
- net Net-(D3-Pad2): track 18.8 -> 10.7 mm
- net Net-(D2-Pad2): track 18.8 -> 10.7 mm
- net Net-(D1-Pad2): track 18.8 -> 10.7 mm
Changed lines of the file:
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@@
 (kicad_pcb (version 4) (host pcbnew 4.0.6)
   (general
-    (links 28)
-    (no_connects 20)
+    (links 25)
+    (no_connects 5)
     (area 110.922999 72.949999 179.653001 126.440001)
     (thickness 1.6)
@@
     (zones 0)
     (modules 20)
-    (nets 45)
+    (nets 48)
   )
   (page A4)
@@
   (net 43 "Net-(J1-Pad3)")
   (net 44 "Net-(J3-Pad1)")
+  (net 45 "Net-(Q1-Pad1)")
+  (net 46 "Net-(Q2-Pad1)")
+  (net 47 "Net-(Q3-Pad1)")
   (net_class Default "This is the default net class."
     (clearance 0.2)
@@
     (add_net "Net-(P7-Pad1)")
     (add_net "Net-(P8-Pad1)")
+    (add_net "Net-(Q1-Pad1)")
+    (add_net "Net-(Q2-Pad1)")
+    (add_net "Net-(Q3-Pad1)")
   )
   (module Socket_Arduino_Uno:Socket_Strip_Arduino_1x08 locked (layer F.Cu)
@@
     (fp_line (start 7.79 -2.75) (end -2.71 -2.75) (layer F.CrtYd) (width 0.05))
     (pad 1 thru_hole rect (at 0 0) (size 1.8 1.8) (drill 1) (layers *.Cu *.Mask)
-      (net 39 "Net-(D1-Pad2)"))
+      (net 45 "Net-(Q1-Pad1)"))
     (pad 2 thru_hole oval (at 2.54 0) (size 1.8 1.8) (drill 1) (layers *.Cu *.Mask)
       (net 36 "Net-(J2-Pad4)"))
@@
     (fp_line (start 7.79 -2.75) (end -2.71 -2.75) (layer F.CrtYd) (width 0.05))
     (pad 1 thru_hole rect (at 0 0) (size 1.8 1.8) (drill 1) (layers *.Cu *.Mask)
-      (net 40 "Net-(D2-Pad2)"))
+      (net 46 "Net-(Q2-Pad1)"))
     (pad 2 thru_hole oval (at 2.54 0) (size 1.8 1.8) (drill 1) (layers *.Cu *.Mask)
       (net 37 "Net-(J2-Pad3)"))
@@
     (fp_line (start 7.79 -2.75) (end -2.71 -2.75) (layer F.CrtYd) (width 0.05))
     (pad 1 thru_hole rect (at 0 0) (size 1.8 1.8) (drill 1) (layers *.Cu *.Mask)
-      (net 41 "Net-(D3-Pad2)"))
+      (net 47 "Net-(Q3-Pad1)"))
     (pad 2 thru_hole oval (at 2.54 0) (size 1.8 1.8) (drill 1) (layers *.Cu *.Mask)
       (net 38 "Net-(J2-Pad2)"))
@@
     (fp_line (start 8.7 -1.6) (end -1.05 -1.6) (layer F.CrtYd) (width 0.05))
     (pad 1 thru_hole circle (at 0 0 180) (size 1.6 1.6) (drill 0.8) (layers *.Cu *.Mask)
-      (net 39 "Net-(D1-Pad2)"))
+      (net 45 "Net-(Q1-Pad1)"))
     (pad 2 thru_hole oval (at 7.62 0 180) (size 1.6 1.6) (drill 0.8) (layers *.Cu *.Mask)
       (net 6 "/5(**)"))
@@
     (fp_line (start 8.7 -1.6) (end -1.05 -1.6) (layer F.CrtYd) (width 0.05))
     (pad 1 thru_hole circle (at 0 0 180) (size 1.6 1.6) (drill 0.8) (layers *.Cu *.Mask)
-      (net 40 "Net-(D2-Pad2)"))
+      (net 46 "Net-(Q2-Pad1)"))
     (pad 2 thru_hole oval (at 7.62 0 180) (size 1.6 1.6) (drill 0.8) (layers *.Cu *.Mask)
       (net 3 "/9(**)"))
@@
     (fp_line (start 8.7 -1.6) (end -1.05 -1.6) (layer F.CrtYd) (width 0.05))
     (pad 1 thru_hole circle (at 0 0 180) (size 1.6 1.6) (drill 0.8) (layers *.Cu *.Mask)
-      (net 41 "Net-(D3-Pad2)"))
+      (net 47 "Net-(Q3-Pad1)"))
     (pad 2 thru_hole oval (at 7.62 0 180) (size 1.6 1.6) (drill 0.8) (layers *.Cu *.Mask)
       (net 12 "/10(**/SS)"))
@@
   (segment (start 170.744 102.409) (end 172.974 102.409) (width 0.25) (layer F.Cu) (net 38))
   (segment (start 143.51 112.649) (end 154.178 112.649) (width 0.25) (layer F.Cu) (net 39))
-  (segment (start 135.382 112.649) (end 143.51 112.649) (width 0.25) (layer F.Cu) (net 39))
   (segment (start 143.51 105.029) (end 154.178 105.029) (width 0.25) (layer F.Cu) (net 40))
-  (segment (start 135.382 105.029) (end 143.51 105.029) (width 0.25) (layer F.Cu) (net 40))
   (segment (start 143.51 97.409) (end 154.178 97.409) (width 0.25) (layer F.Cu) (net 41))
-  (segment (start 135.382 97.409) (end 143.51 97.409) (width 0.25) (layer F.Cu) (net 41))
+  (segment (start 135.382 112.649) (end 143.51 112.649) (width 0.25) (layer F.Cu) (net 45))
+  (segment (start 135.382 105.029) (end 143.51 105.029) (width 0.25) (layer F.Cu) (net 46))
+  (segment (start 135.382 97.409) (end 143.51 97.409) (width 0.25) (layer F.Cu) (net 47))
 )
